File: authbox-relay-driver.kicad_sch (KiCad schematic)
At the start: 11 parts, among them J1 GPIO, J2 Screw_Terminal_01x12, Q2 BC846, Q3 BC846, U2 MCP1415

Commit message: Miscellaneous fixes: * Change to KiCad 8.0. * Modify the cutouts on the board to accomodate a different layout of the   PoE hat (which sits below.) * Transfer the customized footprints into a project-specific "hat-library"   footprints library, rather than leave them with local edits. * Change the mounting holes from through-plated to NPTH.
Parts:
- C4, C5: footprint Capacitor_SMD:C_0603_1608Metric_Pad0.99x1.00mm_HandSolder -> Capacitor_SMD:C_0603_1608Metric_Pad1.08x0.95mm_HandSolder
- J1: footprint Connector_PinSocket_2.54mm:PinSocket_2x20_P2.54mm_Vertical -> hat-library:PinSocket_2x20_P2.54mm_Vertical
- J2: footprint Connector_Phoenix_MC:PhoenixContact_MC_1,5_12-G-3.5_1x12_P3.50mm_Horizontal -> hat-library:PhoenixContact_MC_1,5_12-G-3.5_1x12_P3.50mm_Horizontal
- R1, R11, R12, R2: footprint Resistor_SMD:R_0603_1608Metric_Pad0.99x1.00mm_HandSolder -> Resistor_SMD:R_0603_1608Metric_Pad0.98x0.95mm_HandSolder
- U2: footprint Package_TO_SOT_SMD:SOT-23-5 -> hat-library:SOT-23-5
Connections:
- no-connect marks 0 -> 22
Other:
- added sheet Mechanical (mechanical.kicad_sch)
