File: current-sense.kicad_sch (KiCad schematic)
At the start: 11 parts, among them Q1 2N7002L

Commit message: Miscellaneous fixes: * Change to KiCad 8.0. * Modify the cutouts on the board to accomodate a different layout of the   PoE hat (which sits below.) * Transfer the customized footprints into a project-specific "hat-library"   footprints library, rather than leave them with local edits. * Change the mounting holes from through-plated to NPTH.
Parts:
- removed RV1: 5M, Potentiometer_THT:Potentiometer_Bourns_3386P_Vertical, symbol Device:R_POT_TRIM
- added RV1: 5M, hat-library:Potentiometer_Bourns_3386P_Vertical, symbol Device:R_Potentiometer_Trim
- C1, C2: footprint Capacitor_SMD:C_0603_1608Metric_Pad0.99x1.00mm_HandSolder -> Capacitor_SMD:C_0603_1608Metric_Pad1.08x0.95mm_HandSolder
- D4: footprint Diode_SMD:Diode_Bridge_Diotec_ABS -> hat-library:Diode_Bridge_Diotec_ABS
- D6: footprint LED_SMD:LED_0603_1608Metric_Pad0.82x1.00mm_HandSolder -> LED_SMD:LED_0603_1608Metric_Pad1.05x0.95mm_HandSolder
- R4, R5, R6, R7: footprint Resistor_SMD:R_0603_1608Metric_Pad0.99x1.00mm_HandSolder -> Resistor_SMD:R_0603_1608Metric_Pad0.98x0.95mm_HandSolder
Connections:
- net GND: now also RV1.1
- net at C1.1, D2.1 (K), D4.1 (+)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: now also RV1.2, RV1.3
